Commit message: kinectモデルにprefix引数を追加
prefix引数を設定することで
prefix + topic名
となる

File: two_kinect_description/urdf/sensor/kinect.gazebo.xacro (robot description, xacro)
@@ -2,5 +2,5 @@
 <robot xmlns:xacro="http://ros.org/wiki/xacro">
   <xacro:include filename="$(find two_kinect_description)/urdf/common.xacro" />
-  <xacro:macro name="kinect_gazebo" params="name">
+  <xacro:macro name="kinect_gazebo" params="name suffix">
     <gazebo reference="${name}_link">
       <mu1>0.2</mu1>
@@ -29,5 +29,5 @@
         </camera>
         <plugin name="${name}_camera_controller" filename="libgazebo_ros_openni_kinect.so">
-          <cameraName>kinect2/hd</cameraName>
+          <cameraName>${suffix}/kinect2/hd</cameraName>
           <alwaysOn>true</alwaysOn>
           <updateRate>30</updateRate>
@@ -70,5 +70,5 @@
         </camera>
         <plugin name="${name}_camera_controller" filename="libgazebo_ros_openni_kinect.so">
-          <cameraName>kinect2/qhd</cameraName>
+          <cameraName>${suffix}/kinect2/qhd</cameraName>
           <alwaysOn>true</alwaysOn>
           <updateRate>30</updateRate>
@@ -111,5 +111,5 @@
         </camera>
         <plugin name="${name}_camera_controller" filename="libgazebo_ros_openni_kinect.so">
-          <cameraName>kinect2/sd</cameraName>
+          <cameraName>${suffix}/kinect2/sd</cameraName>
           <alwaysOn>true</alwaysOn>
           <updateRate>30</updateRate>
