Commit message: jointもxacroでマクロ化
suffixはnamespaceの役割を果たしておりtfとトピック名の始めに付加される

File: two_kinect_description/urdf/sensor/kinect.urdf.xacro (robot description, xacro)
@@ -1,5 +1,5 @@
 <?xml version="1.0"?>
 <robot xmlns:xacro="http://ros.org/wiki/xacro">
-<xacro:macro name="kinect2_link_box_v0" params="name">
+  <xacro:macro name="kinect2_link_box_v0" params="name">
     <link name="${name}">
       <visual>
@@ -22,4 +22,21 @@
       </inertial>
     </link>
-</xacro:macro>
+  </xacro:macro>
+  <xacro:macro name="kinect_joints" params="suffix rpy xyz">
+    <xacro:kinect2_link_box_v0 name="${suffix}/kinect2_link"/>
+    <link name="${suffix}/kinect2_rgb_optical_frame"/>
+    <!-- Joint -->
+    <joint name="${suffix}/joint_kinect2" type="fixed">
+      <origin rpy="${rpy}" xyz="${xyz}"/>
+      <parent link="world"/>
+      <child link="${suffix}/kinect2_link"/>
+    </joint>
+    <joint name="${suffix}/joint_rgb_kinect2" type="fixed">
+      <origin rpy="${M_PI/2} ${M_PI} ${M_PI/2}"/>
+      <parent link="${suffix}/kinect2_link"/>
+      <child link="${suffix}/kinect2_rgb_optical_frame"/>
+    </joint>
+    <!-- Gazebo -->
+    <xacro:kinect_gazebo name="${suffix}/kinect2" suffix="${suffix}"/>
+  </xacro:macro>
 </robot>
