Commit message: なんとかひとつキネクトが出るようになりました

File: two_kinect_description/robots/multi_kinectv2.urdf.xacro (robot description, xacro)
@@ -1,10 +1,12 @@
 <?xml version="1.0"?>
-<robot name="sia5" xmlns:xacro="http://ros.org/wiki/xacro">
+<robot name="kinect2" xmlns:xacro="http://ros.org/wiki/xacro">
   <!-- File Include -->
+  <xacro:include filename="$(find two_kinect_description)/urdf/common.xacro" />
+  <xacro:include filename="$(find two_kinect_description)/urdf/materials.xacro"/>
   <xacro:include filename="$(find two_kinect_description)/urdf/sensor/kinect.urdf.xacro"/>
   <xacro:include filename="$(find two_kinect_description)/urdf/sensor/kinect.gazebo.xacro"/>
   <!-- add Kinect V2 -->
   <!-- Link -->
-  <link name="world" />
+  <link name="world"/>
   <xacro:kinect2_link_box_v0 name="kinect2_link"/>
   <link name="kinect2_rgb_optical_frame"/>
@@ -16,7 +18,7 @@
   </joint>
   <joint name="joint_rgb_kinect2" type="fixed">
-	<origin rpy="${M_PI/2} ${M_PI} ${M_PI/2}"/>
-	<parent link="kinect2_link"/>
-	<child link="kinect2_rgb_optical_frame"/>
+    <origin rpy="${M_PI/2} ${M_PI} ${M_PI/2}"/>
+    <parent link="kinect2_link"/>
+    <child link="kinect2_rgb_optical_frame"/>
   </joint>
   <!-- Gazebo -->

File: two_kinect_description/urdf/sensor/kinect.gazebo.xacro (robot description, xacro)
@@ -2,31 +2,31 @@
 <robot xmlns:xacro="http://ros.org/wiki/xacro">
   <xacro:include filename="$(find two_kinect_description)/urdf/common.xacro" />
-  <xacro:macro name="two_kinect_gazebo" params="name">
-	<gazebo reference="${name}_link">
-	  <mu1>0.2</mu1>
-	  <mu2>0.2</mu2>
-	  <material>Gazebo/Black</material>
-	  <!-- hd -->
+  <xacro:macro name="kinect_gazebo" params="name">
+    <gazebo reference="${name}_link">
+      <mu1>0.2</mu1>
+      <mu2>0.2</mu2>
+      <material>Gazebo/Black</material>
+      <!-- hd -->
       <sensor type="depth" name="${name}">
-		<always_on>true</always_on>
-		<update_rate>30.0</update_rate>
-		<camera>
+        <always_on>true</always_on>
+        <update_rate>30.0</update_rate>
+        <camera>
           <horizontal_fov>${84.1*M_PI/180.0}</horizontal_fov>
           <image>
-			<format>R8G8B8</format>
-			<width>512</width>
-			<height>424</height>
+        <format>R8G8B8</format>
+        <width>512</width>
+        <height>424</height>
           </image>
           <clip>
-			<near>0.05</near>
-			<far>4.5</far>
+        <near>0.05</near>
+        <far>4.5</far>
           </clip>
-		  <noise>
-			<type>gaussian</type>
-			<mean>0.0</mean>
-			<stddev>0.005</stddev>
-		  </noise>
-		</camera>
-		<plugin name="${name}_camera_controller" filename="libgazebo_ros_openni_kinect.so">
+          <noise>
+            <type>gaussian</type>
+            <mean>0.0</mean>
+            <stddev>0.005</stddev>
+          </noise>
+        </camera>
+        <plugin name="${name}_camera_controller" filename="libgazebo_ros_openni_kinect.so">
           <cameraName>kinect2/hd</cameraName>
           <alwaysOn>true</alwaysOn>
@@ -45,29 +45,29 @@
           <distortion_t2>0.0</distortion_t2>
           <pointCloudCutoff>0.05</pointCloudCutoff>
-		  <pointCloudCutoffMax>4.5</pointCloudCutoffMax>
-		</plugin>
+          <pointCloudCutoffMax>4.5</pointCloudCutoffMax>
+        </plugin>
       </sensor>
-	  <!-- qhd -->
+      <!-- qhd -->
       <sensor type="depth" name="${name}">
-		<always_on>true</always_on>
-		<update_rate>30.0</update_rate>
-		<camera>
+        <always_on>true</always_on>
+        <update_rate>30.0</update_rate>
+        <camera>
           <horizontal_fov>${84.1*M_PI/180.0}</horizontal_fov>
           <image>
-			<format>R8G8B8</format>
-			<width>512</width>
-			<height>424</height>
+            <format>R8G8B8</format>
+            <width>512</width>
+            <height>424</height>
           </image>
           <clip>
-			<near>0.05</near>
-			<far>4.5</far>
+            <near>0.05</near>
+            <far>4.5</far>
           </clip>
-		  <noise>
-			<type>gaussian</type>
-			<mean>0.0</mean>
-			<stddev>0.005</stddev>
-		  </noise>
-		</camera>
-		<plugin name="${name}_camera_controller" filename="libgazebo_ros_openni_kinect.so">
+          <noise>
+            <type>gaussian</type>
+            <mean>0.0</mean>
+            <stddev>0.005</stddev>
+          </noise>
+        </camera>
+        <plugin name="${name}_camera_controller" filename="libgazebo_ros_openni_kinect.so">
           <cameraName>kinect2/qhd</cameraName>
           <alwaysOn>true</alwaysOn>
@@ -86,29 +86,29 @@
           <distortion_t2>0.0</distortion_t2>
           <pointCloudCutoff>0.05</pointCloudCutoff>
-		  <pointCloudCutoffMax>4.5</pointCloudCutoffMax>
-		</plugin>
+          <pointCloudCutoffMax>4.5</pointCloudCutoffMax>
+        </plugin>
       </sensor>
 	  <!-- sd -->
       <sensor type="depth" name="${name}">
-		<always_on>true</always_on>
-		<update_rate>30.0</update_rate>
-		<camera>
+        <always_on>true</always_on>
+        <update_rate>30.0</update_rate>
+        <camera>
           <horizontal_fov>${84.1*M_PI/180.0}</horizontal_fov>
           <image>
-			<format>R8G8B8</format>
-			<width>512</width>
-			<height>424</height>
+            <format>R8G8B8</format>
+            <width>512</width>
+            <height>424</height>
           </image>
           <clip>
-			<near>0.05</near>
-			<far>4.5</far>
+          <near>0.05</near>
+          <far>4.5</far>
           </clip>
-		  <noise>
-			<type>gaussian</type>
-			<mean>0.0</mean>
-			<stddev>0.005</stddev>
-		  </noise>
-		</camera>
-		<plugin name="${name}_camera_controller" filename="libgazebo_ros_openni_kinect.so">
+          <noise>
+            <type>gaussian</type>
+            <mean>0.0</mean>
+            <stddev>0.005</stddev>
+          </noise>
+        </camera>
+        <plugin name="${name}_camera_controller" filename="libgazebo_ros_openni_kinect.so">
           <cameraName>kinect2/sd</cameraName>
           <alwaysOn>true</alwaysOn>
@@ -127,8 +127,8 @@
           <distortion_t2>0.0</distortion_t2>
           <pointCloudCutoff>0.05</pointCloudCutoff>
-		  <pointCloudCutoffMax>4.5</pointCloudCutoffMax>
-		</plugin>
+          <pointCloudCutoffMax>4.5</pointCloudCutoffMax>
+        </plugin>
       </sensor>
-	</gazebo>
+    </gazebo>
   </xacro:macro>
 </robot>

File: two_kinect_description/urdf/sensor/kinect.urdf.xacro (robot description, xacro)
@@ -4,5 +4,5 @@
     <link name="${name}">
       <visual>
-		<material name="black"/>
+        <material name="black"/>
         <geometry>
           <mesh filename="package://two_kinect_description/meshes/sensor/visual/COLLADA/kinectv2.stl"/>
@@ -10,7 +10,7 @@
       </visual>
       <collision>
-		<origin xyz="0 0 0.041"/>
+        <origin xyz="0 0 0.041"/>
         <geometry>
-		  <box size="0.065 0.25 0.082"/>
+          <box size="0.065 0.25 0.082"/>
         </geometry>
       </collision>
@@ -18,6 +18,6 @@
         <mass value="0.935"/>
         <inertia ixx="0.0053937" ixy="0" ixz="0"
-				 iyy="0.00085311" iyz="0"
-				 izz="0.00519899" />
+                 iyy="0.00085311" iyz="0"
+                 izz="0.00519899" />
       </inertial>
     </link>

Commit message: kinectを2つ出すように定義

File: two_kinect_description/robots/multi_kinectv2.urdf.xacro (robot description, xacro)
@@ -9,18 +9,5 @@
   <!-- Link -->
   <link name="world"/>
-  <xacro:kinect2_link_box_v0 name="kinect2_link"/>
-  <link name="kinect2_rgb_optical_frame"/>
-  <!-- Joint -->
-  <joint name="joint_kinect2" type="fixed">
-    <origin rpy="0 ${10*M_PI/180} ${M_PI}" xyz="1.05024 0 0.3195"/>
-    <parent link="world"/>
-    <child link="kinect2_link"/>
-  </joint>
-  <joint name="joint_rgb_kinect2" type="fixed">
-    <origin rpy="${M_PI/2} ${M_PI} ${M_PI/2}"/>
-    <parent link="kinect2_link"/>
-    <child link="kinect2_rgb_optical_frame"/>
-  </joint>
-  <!-- Gazebo -->
-  <xacro:kinect_gazebo name="kinect2"/>
+  <xacro:kinect_joints suffix="/kinect_first" rpy="0 ${10*M_PI/180} ${M_PI}" xyz="0 1 0.5"/>
+  <xacro:kinect_joints suffix="/kinect_second" rpy="0 ${10*M_PI/180} ${M_PI}" xyz="0 -1 0.5"/>
 </robot>

Commit message: 検証用環境の完成！

File: two_kinect_description/robots/multi_kinectv2.urdf.xacro (robot description, xacro)
@@ -9,4 +9,10 @@
   <!-- Link -->
   <link name="world"/>
+  <link name="virtual_kinect2_frame"/>
+  <joint name="virtual_kinect_joint" type="fixed">
+    <origin rpy="0 0 0" xyz="0 1 0.5"/>
+    <parent link="world"/>
+    <child link="virtual_kinect2_frame"/>
+  </joint>
   <xacro:kinect_joints suffix="/kinect_first" rpy="0 ${10*M_PI/180} 0" xyz="0 0 0.5"/>
   <xacro:kinect_joints suffix="/kinect_second" rpy="0 ${10*M_PI/180} ${1.5*M_PI}" xyz="1 1 0.5"/>

Commit message: 3つキネクトを出して試しています

File: two_kinect_description/robots/multi_kinectv2.urdf.xacro (robot description, xacro)
@@ -9,11 +9,12 @@
   <!-- Link -->
   <link name="world"/>
-  <link name="virtual_kinect2_frame"/>
+  <link name="virtual_kinect2_link"/>
   <joint name="virtual_kinect_joint" type="fixed">
-    <origin rpy="0 0 0" xyz="0 1 0.5"/>
+    <origin rpy="0 0 0" xyz="-1 0 0.5"/>
     <parent link="world"/>
-    <child link="virtual_kinect2_frame"/>
+    <child link="virtual_kinect2_link"/>
   </joint>
-  <xacro:kinect_joints suffix="/kinect_first" rpy="0 ${10*M_PI/180} 0" xyz="0 0 0.5"/>
-  <xacro:kinect_joints suffix="/kinect_second" rpy="0 ${10*M_PI/180} ${1.5*M_PI}" xyz="1 1 0.5"/>
+  <xacro:kinect_joints suffix="/kinect_first" rpy="0 0 -${120*M_PI/180}" xyz="1 1.7320 0.5"/>
+  <xacro:kinect_joints suffix="/kinect_second" rpy="0 0 ${120*M_PI/180}" xyz="1 -1.7320 0.5"/>
+  <xacro:kinect_joints suffix="/kinect_third" rpy="0 0 0" xyz="-2 0 0.5"/>
 </robot>
