Commit message: パッケージ名を変更したので，それに伴う内容修正

File: multi_kinect_description/urdf/sensor/kinect.gazebo.xacro (robot description, xacro)
@@ -1,5 +1,5 @@
 <?xml version="1.0"?>
 <robot xmlns:xacro="http://ros.org/wiki/xacro">
-  <xacro:include filename="$(find two_kinect_description)/urdf/common.xacro" />
+  <xacro:include filename="$(find multi_kinect_description)/urdf/common.xacro" />
   <xacro:macro name="kinect_gazebo" params="name suffix">
     <gazebo reference="${name}_link">

File: multi_kinect_description/urdf/sensor/kinect.urdf.xacro (robot description, xacro)
@@ -6,5 +6,5 @@
         <material name="black"/>
         <geometry>
-          <mesh filename="package://two_kinect_description/meshes/sensor/visual/COLLADA/kinectv2.stl"/>
+          <mesh filename="package://multi_kinect_description/meshes/sensor/visual/COLLADA/kinectv2.stl"/>
         </geometry>
       </visual>
